Commit message: Camera add

File: ur_description/urdf/ur.gazebo.xacro (robot description, xacro)
@@ -23,4 +23,44 @@
       <selfCollide>true</selfCollide>
     </gazebo>
+  <!-- camera -->
+  <gazebo reference="camera_link">
+    <sensor type="camera" name="camera1">
+      <update_rate>30.0</update_rate>
+      <camera name="head">
+        <horizontal_fov>1.3962634</horizontal_fov>
+        <image>
+          <width>800</width>
+          <height>800</height>
+          <format>R8G8B8</format>
+        </image>
+        <clip>
+          <near>0.02</near>
+          <far>300</far>
+        </clip>
+        <noise>
+          <type>gaussian</type>
+          <!-- Noise is sampled independently per pixel on each frame.
+          That pixel's noise value is added to each of its color
+          channels, which at that point lie in the range [0,1]. -->
+          <mean>0.0</mean>
+          <stddev>0.007</stddev>
+        </noise>
+      </camera>
+      <plugin name="camera_controller" filename="libgazebo_ros_camera.so">
+        <alwaysOn>true</alwaysOn>
+        <updateRate>0.0</updateRate>
+        <cameraName>rrbot/camera1</cameraName>
+        <imageTopicName>image_raw</imageTopicName>
+        <cameraInfoTopicName>camera_info</cameraInfoTopicName>
+        <frameName>camera_link</frameName>
+        <hackBaseline>0.07</hackBaseline>
+        <distortionK1>0.0</distortionK1>
+        <distortionK2>0.0</distortionK2>
+        <distortionK3>0.0</distortionK3>
+        <distortionT1>0.0</distortionT1>
+        <distortionT2>0.0</distortionT2>
+      </plugin>
+    </sensor>
+  </gazebo>
   </xacro:macro>
 </robot>

File: ur_description/urdf/ur3.urdf.xacro (robot description, xacro)
@@ -6,4 +6,10 @@
   <xacro:include filename="$(find ur_description)/urdf/ur.transmission.xacro" />
   <xacro:include filename="$(find ur_description)/urdf/ur.gazebo.xacro" />
+  <!-- Camera -->
+  <xacro:include filename="$(find ur_description)/urdf/camera.xacro" />
+  <!-- Constants -->
+  <xacro:property name="PI" value="3.1415926535897931"/>
+  <!-- Camera -->
+  <xacro:property name="camera_link" value="0.05" /> <!-- Size of square 'camera' box -->
    <xacro:macro name="cylinder_inertial" params="radius length mass *origin">
     <inertial>
@@ -335,3 +341,4 @@
     </joint>
   </xacro:macro>
+  <xacro:camera_body/>
 </robot>
