Commit message: Camara en otra pos

File: ur_description/urdf/camera.xacro (robot description, xacro)
@@ -4,6 +4,6 @@
 		<joint name="camera_joint" type="fixed">
 			<axis xyz="0 1 0" />
-			<origin xyz="0.5 -0.2 0.2" rpy="0 0 ${-PI/2}"/>
-			<parent link="wrist_3_link"/>
+			<origin xyz="-0.08 0 0" rpy="0 0 ${PI/2}"/>
+			<parent link="wrist_2_link"/>
 			<child link="camera_link"/>
 		</joint>
