Commit message: Changes panel.

File: panel_description/urdf/button.xacro (robot description, xacro)
@@ -1,5 +1,11 @@
 <?xml version="1.0" ?>
 <robot xmlns:xacro="http://www.ros.org/wiki/xacro">
-	<xacro:macro name="button" params="">
+	<xacro:macro name="button" params="link_sector x y">
+		<!-- SECTOR_BUTTONS TO CYLINDER JOINT -->
+		<joint name="lid_spring_joint" type="fixed">
+			<parent link="${link_sector}"/>
+			<child link="spring_link"/>
+			<origin xyz="-0.15 0 0" rpy="0 0 ${PI}"/>
+		</joint>
 		<!-- BUTTON LID -->
 		<link name='lid_link'>
