Commit message: Archivos launch para RViz y Gazebo.

File: panel_description/urdf/box.xacro (robot description, xacro)
@@ -6,5 +6,5 @@
 			<parent link="base_footprint"/>
 			<child link="box_link"/>
-			<origin xyz="-0.15 0 0" rpy="0 0 ${PI}"/>
+			<origin xyz="0 0 0" rpy="0 0 0"/>
 		</joint>
 		<link name='box_link'>
@@ -12,5 +12,5 @@
 				<origin xyz="0 0 0"	rpy="0 0 0"/>
 				<geometry>
-					<mesh filename="package://panel_description/meshes/visual/lid.stl" scale="${scale_XYZ} ${scale_XYZ} ${scale_XYZ}"/>
+					<mesh filename="package://panel_description/meshes/visual/box.stl" scale="${scale_XYZ} ${scale_XYZ} ${scale_XYZ}"/>
 				</geometry>
 			</collision>
@@ -18,5 +18,5 @@
 				<origin xyz="0 0 0"	rpy="0 0 0"/>
 				<geometry>
-					<mesh filename="package://panel_description/meshes/visual/lid.stl" scale="${scale_XYZ} ${scale_XYZ} ${scale_XYZ}"/>
+					<mesh filename="package://panel_description/meshes/visual/box.stl" scale="${scale_XYZ} ${scale_XYZ} ${scale_XYZ}"/>
 				</geometry>
 			</visual>

File: panel_description/urdf/panel.xacro (robot description, xacro)
@@ -10,14 +10,14 @@
 	<xacro:include filename="$(find panel_description)/urdf/box.xacro" />
 	<!-- sector_buttons -->
-	<xacro:include filename="$(find panel_description)/urdf/sector_buttons.xacro" />
+	<!-- <xacro:include filename="$(find panel_description)/urdf/sector_buttons.xacro" /> -->
 	<!-- sector_extra -->
-	<xacro:include filename="$(find panel_description)/urdf/sector_extra.xacro" />
+	<!-- <xacro:include filename="$(find panel_description)/urdf/sector_extra.xacro" /> -->
 	<!-- sector_switches -->
-	<xacro:include filename="$(find panel_description)/urdf/sector_switches.xacro" />
+	<!-- <xacro:include filename="$(find panel_description)/urdf/sector_switches.xacro" /> -->
 	<!-- Join parts -->
 	<xacro:box/>
-	<xacro:sector_buttons/>
-	<xacro:sector_extra/>
-	<xacro:sector_switches/>
+	<!-- <xacro:sector_buttons/> -->
+	<!-- <xacro:sector_extra/> -->
+	<!-- <xacro:sector_switches/> -->
 	<!-- <xacro:camera_body/> -->
 </robot>

File: panel_description/urdf/properties.xacro (robot description, xacro)
@@ -9,5 +9,9 @@
 	<xacro:property name="camera_link" value="0.05" /> <!-- Size of square 'camera' box -->
 	<!-- Panel properties -->
-	<!-- Button properties -->
+	<xacro:property name="boxMass" value="1"/>
+	<xacro:property name="boxWidth" value="0.4327"/>
+	<xacro:property name="boxLength" value="0.72"/>
+	<xacro:property name="boxHeight" value="0.174"/>
+	<!-- box properties -->
 	<xacro:property name="buttonMass" value="10"/>
 	<xacro:property name="buttonWidth" value="0.4327"/>

Commit message: switch xacro

File: panel_description/urdf/box.xacro (robot description, xacro)
@@ -27,4 +27,5 @@
 			</inertial>
 		</link>
+		<!-- <xacro:switch parent_sector_link ="box_link"  child_link= "switch" x="0" y="0"/> -->
 	</xacro:macro>
 </robot>

File: panel_description/urdf/panel.xacro (robot description, xacro)
@@ -9,4 +9,6 @@
 	<!-- box -->
 	<xacro:include filename="$(find panel_description)/urdf/box.xacro" />
+	<xacro:include filename="$(find panel_description)/urdf/switch.xacro" />
+	<xacro:include filename="$(find panel_description)/urdf/sector_switches.xacro" />
 	<!-- sector_buttons -->
 	<!-- <xacro:include filename="$(find panel_description)/urdf/sector_buttons.xacro" /> -->
@@ -16,8 +18,10 @@
 	<!-- <xacro:include filename="$(find panel_description)/urdf/sector_switches.xacro" /> -->
 	<!-- Join parts -->
-	<xacro:box/>
+	<!---<xacro:box/> -->
 	<!-- <xacro:sector_buttons/> -->
 	<!-- <xacro:sector_extra/> -->
-	<!-- <xacro:sector_switches/> -->
+	<xacro:sector_switches/>
 	<!-- <xacro:camera_body/> -->
+	<!--<link name="base_footprint" />
+	<xacro:switch parent_sector_link ="base_footprint"  child_link= "switch" x="0" y="0"/>-->
 </robot>

File: panel_description/urdf/properties.xacro (robot description, xacro)
@@ -20,4 +20,36 @@
 	<!-- Pot properties -->
 	<!-- Switch properties -->
+	<!-- Switch box properties-->
+	<xacro:property name="switchboxMass" value="0.770"/>
+	<xacro:property name="switchboxWidth" value="0.320"/>
+	<xacro:property name="switchboxLength" value="0.380"/>
+	<xacro:property name="switchboxHeight" value="0.020"/>
+	<!-- enclosure properties -->
+	<xacro:property name="enclosureMass" value="0.005"/>
+	<xacro:property name="enclosureWidth" value="0.019"/>
+	<xacro:property name="enclosureLength" value="0.030"/>
+	<xacro:property name="enclosureHeight" value="0.026"/>
+	<!-- Base properties -->
+	<xacro:property name="baseMass" value="0.016"/>
+	<xacro:property name="baseWidth" value="0.010"/>
+	<xacro:property name="baseLength" value="0.010"/>
+	<xacro:property name="baseHeight" value="0.070"/>
+	<!-- Triangle properties -->
+	<xacro:property name="triangleMass" value="0.010"/>
+	<xacro:property name="triangleWidth" value="0.010"/>
+	<xacro:property name="triangleLength" value="0.02"/>
+	<xacro:property name="triangleHeight" value="0.010"/>
+	<!-- Trigger properties -->
+	<xacro:property name="triggerMass" value="0.002"/>
+	<xacro:property name="triggerRadio" value="0.003"/>
+	<xacro:property name="triggerHeight" value="0.011"/>
+	<!-- Spring properties -->
+	<xacro:property name="springMass" value="0.003"/>
+	<xacro:property name="springRadio" value="0.00275"/>
+	<xacro:property name="springHeight" value="0.005"/>
+	<!-- Lever properties -->
+	<xacro:property name="leverMass" value="0.008"/>
+	<xacro:property name="leverRadio" value="0.0045"/>
+	<xacro:property name="leverHeight" value="0.030"/>
 	<!-- Pot properties -->
 	<!-- Pot properties -->

File: panel_description/urdf/sector_switches.xacro (robot description, xacro)
@@ -1,32 +1,43 @@
 <?xml version="1.0"?>
-<robot name="rex" xmlns:xacro="http://www.ros.org/wiki/xacro">
-	<joint name="sector_switch_joint" type="fixed">
-		<parent link="box_link"/>
-		<child link="sector_switch_link"/>
-		<origin xyz="-0.15 0 0" rpy="0 0 ${PI}"/>
-	</joint>
-	<link name='sector_switch_link'>
-		<collision>
-			<origin xyz="0 0 0"	rpy="0 0 0"/>
-			<geometry>
-				<mesh filename="package://panel_description/meshes/visual/lid.stl" scale="${scale_XYZ} ${scale_XYZ} ${scale_XYZ}"/>
-			</geometry>
-		</collision>
-		<visual>
-			<origin xyz="0 0 0"	rpy="0 0 0"/>
-			<geometry>
-				<mesh filename="package://panel_description/meshes/visual/lid.stl" scale="${scale_XYZ} ${scale_XYZ} ${scale_XYZ}"/>
-			</geometry>
-		</visual>
-		<inertial>
-			<origin xyz="0 0 0"	rpy="0 0 0"/>
-			<mass value="${boxMass}"/>
-			<xacro:box_inertia m="${boxMass}" x="${boxWidth}" y="${boxLength}" z="${boxHeight}" />
-		</inertial>
-	</link>
-	<!-- Inertia matrices -->
-	<xacro:include filename="$(find panel_description)/urdf/switch.xacro" />
-	<!-- Join parts -->
-	<xacro:switch link_sector="sector_switch_link switch_1_joint" x="0.0" y="0.0" />
-	<xacro:switch link_sector="sector_switch_link switch_2_joint" x="0.0" y="0.0" />
+<robot xmlns:xacro="http://www.ros.org/wiki/xacro">
+	<xacro:macro name="sector_switches" params="">
+		<link name="base_footprint"/>
+		<joint name="sector_switch_joint" type="fixed">
+			<parent link="base_footprint"/>
+			<child link="sector_switch_link"/>
+			<origin xyz="0 0 0" rpy="0 0 0"/>
+		</joint>
+		<link name="sector_switch_link">
+			<collision>
+				<origin xyz="0 0 0"	rpy="0 0 0"/>
+				<geometry>
+					<mesh filename="package://panel_description/meshes/collisions/sector_switch.stl" scale="${scale_XYZ} ${scale_XYZ} ${scale_XYZ}"/>
+				</geometry>
+			</collision>
+			<visual>
+				<origin xyz="0 0 0"	rpy="0 0 0"/>
+				<geometry>
+					<mesh filename="package://panel_description/meshes/visual/sector_switch.stl" scale="${scale_XYZ} ${scale_XYZ} ${scale_XYZ}"/>
+				</geometry>
+			</visual>
+			<inertial>
+				<origin xyz="0 0 0"	rpy="0 0 0"/>switch_1_joint
+				<mass value="${switchboxMass}"/>
+				<xacro:box_inertia m="${switchboxMass}" x="${switchboxWidth}" y="${switchboxLength}" z="${switchboxHeight}" />
+			</inertial>
+		</link>
+		<!-- Join parts -->
+		<xacro:switch parent_sector_link ="sector_switch_link"  child_link="switch_1_joint" x="0" y="0"/>
+		<!--<xacro:switch parent_sector_link ="sector_switch_link"  child_link= "switch_2_joint" x="0" y="0"/>
+		<xacro:switch parent_sector_link ="sector_switch_link"  child_link= "switch_3_joint" x="0" y="0"/>
+		<xacro:switch parent_sector_link ="sector_switch_link"  child_link= "switch_4_joint" x="0" y="0"/>
+		<xacro:switch parent_sector_link ="sector_switch_link"  child_link= "switch_5_joint" x="0" y="0"/>
+		<xacro:switch parent_sector_link ="sector_switch_link"  child_link= "switch_6_joint" x="0" y="0"/>
+		<xacro:switch parent_sector_link ="sector_switch_link"  child_link= "switch_7_joint" x="0" y="0"/>
+		<xacro:switch parent_sector_link ="sector_switch_link"  child_link= "switch_8_joint" x="0" y="0"/>
+		<xacro:switch parent_sector_link ="sector_switch_link"  child_link= "switch_9_joint" x="0" y="0"/>
+		<xacro:switch parent_sector_link ="sector_switch_link"  child_link= "switch_10_joint" x="0" y="0"/>
+		<xacro:switch parent_sector_link ="sector_switch_link"  child_link= "switch_11_joint" x="0" y="0"/>
+		<xacro:switch parent_sector_link ="sector_switch_link"  child_link= "switch_12_joint" x="0" y="0"/>-->
+	</xacro:macro>
 </robot>

File: panel_description/urdf/switch.xacro (robot description, xacro)
@@ -2,40 +2,16 @@
 <robot xmlns:xacro="http://www.ros.org/wiki/xacro">
 	<xacro:macro name="switch" params="parent_sector_link child_link x y">
-		<!-- SECTOR_BUTTONS TO CYLINDER JOINT -->
+		<!-- SECTOR_SWITCH TO CYLINDER JOINT -->
 		<joint name="sector_switch_joint" type="fixed">
 			<parent link="${parent_sector_link}"/>
 			<child link="${child_link}"/>
-			<origin xyz="${x} ${y} 0.0" rpy="0 0 0"/>
+			<origin xyz="${x} ${y} 0.1" rpy="0 ${PI/2} 0"/>
 		</joint>
-		<!-- BUTTON LID -->
-		<link name='${child_link}'>
+		<!-- Switch sector LID -->
+		<link name="${child_link}">
 			<collision>
 				<origin xyz="0 0 0"	rpy="0 0 0"/>
 				<geometry>
-					<mesh filename="package://panel_description/meshes/visual/lid.stl" scale="${scale_XYZ} ${scale_XYZ} ${scale_XYZ}"/>
-				</geometry>
-			</collision>
-			<visual>
-				<origin xyz="0 0 0"	rpy="0 0 0"/>
-				<geometry>lid
-					<mesh filename="package://panel_description/meshes/visual/lid.stl" scale="${scale_XYZ} ${scale_XYZ} ${scale_XYZ}"/>
-				</geometry>
-			</visual>
-			<inertial>
-				<origin xyz="0 0 0"	rpy="0 0 0"/>
-				<mass value="${axisMass}"/>
-				<xacro:box_inertia m="${axisMass}" x="${axisWidth}" y="${axisLength}" z="${axisHeight}" />
-			</inertial>
-		</link>
-		<joint name="lid_spring_joint" type="fixed">
-			<parent link="${child_link}"/>
-			<child link="xxxxxxxxx"/>
-			<origin xyz="-0.15 0 0" rpy="0 0 ${PI}"/>
-		</joint>
-		<link name='xxxxxxxxx'>
-			<collision>
-				<origin xyz="0 0 0"	rpy="0 0 0"/>
-				<geometry>
-					<mesh filename="package://panel_description/meshes/visual/lid.stl" scale="${scale_XYZ} ${scale_XYZ} ${scale_XYZ}"/>
+					<mesh filename="package://panel_description/meshes/collisions/Interruptor/Enclosure.stl" scale="${scale_XYZ} ${scale_XYZ} ${scale_XYZ}"/>
 				</geometry>
 			</collision>
@@ -43,11 +19,162 @@
 				<origin xyz="0 0 0"	rpy="0 0 0"/>
 				<geometry>
-					<mesh filename="package://panel_description/meshes/visual/lid.stl" scale="${scale_XYZ} ${scale_XYZ} ${scale_XYZ}"/>
+					<mesh filename="package://panel_description/meshes/visual/Interruptor/Enclosure.stl" scale="${scale_XYZ} ${scale_XYZ} ${scale_XYZ}"/>
 				</geometry>
 			</visual>
 			<inertial>
 				<origin xyz="0 0 0"	rpy="0 0 0"/>
-				<mass value="${axisMass}"/>
-				<xacro:box_inertia m="${axisMass}" x="${axisWidth}" y="${axisLength}" z="${axisHeight}" />
+				<mass value="${enclosureMass}"/>
+				<xacro:box_inertia m="${enclosureMass}" x="${enclosureWidth}" y="${enclosureLength}" z="${enclosureHeight}" />
+			</inertial>
+		</link>
+		<!-- Enclosure TO Base1 JOINT -->
+		<joint name="enclosure_base1_joint" type="fixed">
+			<parent link="${child_link}"/>
+			<child link="base1_link"/>
+			<origin xyz="${-0.0125} ${0.01} ${-0.0125}" rpy="0 ${-3*PI/2} ${-PI/2}"/>
+		</joint>
+		<link name='base1_link'>
+			<collision>
+				<origin xyz="0 0 0"	rpy="0 0 0"/>
+				<geometry>
+					<mesh filename="package://panel_description/meshes/collisions/Interruptor/Base1.stl" scale="${scale_XYZ} ${scale_XYZ} ${scale_XYZ}"/>
+				</geometry>
+			</collision>
+			<visual>
+				<origin xyz="0 0 0"	rpy="0 0 0"/>
+				<geometry>
+					<mesh filename="package://panel_description/meshes/visual/Interruptor/Base1.stl" scale="${scale_XYZ} ${scale_XYZ} ${scale_XYZ}"/>
+				</geometry>
+			</visual>
+			<inertial>
+				<origin xyz="0 0 0"	rpy="0 0 0"/>
+				<mass value="${baseMass}"/>
+				<xacro:box_inertia m="${baseMass}" x="${baseWidth}" y="${baseLength}" z="${baseHeight}" />
+			</inertial>
+		</link>
+		<!-- Enclosure TO Base2 JOINT -->
+		<joint name="enclosure_base2_joint" type="fixed">
+			<parent link="${child_link}"/>
+			<child link="base2_link"/>
+			<origin xyz="${-0.0125} ${0.01} 0.01" rpy="0 0 ${-PI/2}"/>
+		</joint>
+		<link name='base2_link'>
+			<collision>
+				<origin xyz="${-0.01} 0.003 ${-0.005}"	rpy="0 0 0"/>
+				<geometry>
+					<mesh filename="package://panel_description/meshes/collisions/Interruptor/Base2.stl" scale="${scale_XYZ} ${scale_XYZ} ${scale_XYZ}"/>
+				</geometry>
+			</collision>
+			<visual>
+				<origin xyz="0 0 0"	rpy="0 0 0"/>
+				<geometry>
+					<mesh filename="package://panel_description/meshes/visual/Interruptor/Base2.stl" scale="${scale_XYZ} ${scale_XYZ} ${scale_XYZ}"/>
+				</geometry>
+			</visual>
+			<inertial>
+				<origin xyz="0 0 0"	rpy="0 0 0"/>
+				<mass value="${baseMass}"/>
+				<xacro:box_inertia m="${baseMass}" x="${baseWidth}" y="${baseLength}" z="${baseHeight}" />
+			</inertial>
+		</link>
+		<!-- Base1 TO triangle JOINT -->
+		<joint name="base1_triangle_joint" type="fixed">
+			<parent link="base1_link"/>
+			<child link="triangle_link"/>
+			<origin xyz="${-0.01} 0.003 ${-0.005}" rpy="0 0 0"/>
+		</joint>
+		<link name='triangle_link'>
+			<collision>
+				<origin xyz="0 0 0"	rpy="0 0 0"/>
+				<geometry>
+					<mesh filename="package://panel_description/meshes/collisions/Interruptor/Triangle.stl" scale="${scale_XYZ} ${scale_XYZ} ${scale_XYZ}"/>
+				</geometry>
+			</collision>
+			<visual>
+				<origin xyz="0 0 0"	rpy="0 0 0"/>
+				<geometry>
+					<mesh filename="package://panel_description/meshes/visual/Interruptor/Triangle.stl" scale="${scale_XYZ} ${scale_XYZ} ${scale_XYZ}"/>
+				</geometry>
+			</visual>
+			<inertial>
+				<origin xyz="0 0 0"	rpy="0 0 0"/>
+				<mass value="${triangleMass}"/>
+				<xacro:box_inertia m="${triangleMass}" x="${triangleWidth}" y="${triangleLength}" z="${triangleHeight}" />
+			</inertial>
+		</link>
+		<!-- Triangle TO trigger JOINT Existe ligera colision con triangle, solo mover x un poquito (+- 0.001)-->
+		<joint name="triangle_trigger_joint" type="revolute">
+			<parent link="triangle_link"/>
+			<child link="trigger_link"/>
+			<origin xyz="${-0.005} ${0.015} ${0.005}" rpy="${3*PI/2} ${PI/2} ${PI/2}"/>
+			<limit lower="${-PI/4}" upper="${PI/4}" effort="0" velocity="1"/>
+		</joint>
+		<link name='trigger_link'>
+			<collision>
+				<origin xyz="0 0 0"	rpy="0 0 0"/>
+				<geometry>
+					<mesh filename="package://panel_description/meshes/collisions/Interruptor/Trigger.stl" scale="${scale_XYZ} ${scale_XYZ} ${scale_XYZ}"/>
+				</geometry>
+			</collision>
+			<visual>
+				<origin xyz="0 0 0"	rpy="0 0 0"/>
+				<geometry>
+					<mesh filename="package://panel_description/meshes/visual/Interruptor/Trigger.stl" scale="${scale_XYZ} ${scale_XYZ} ${scale_XYZ}"/>
+				</geometry>
+			</visual>
+			<inertial>
+				<origin xyz="0 0 0"	rpy="0 0 0"/>
+				<mass value="${triggerMass}"/>
+				<xacro:cylinder_inertia m="${triggerMass}" r="${triggerRadio}" h="${triggerHeight}" />
+			</inertial>
+		</link>
+<!-- Trigger to spring JOINT -->
+		<joint name="trigger_spring_joint" type="fixed">
+			<parent link="trigger_link"/>
+			<child link="spring_link"/>
+			<origin xyz="0 0 0" rpy="0 0 0"/>
+		</joint>
+		<link name='spring_link'>
+			<collision>
+				<origin xyz="0 0 0"	rpy="0 0 0"/>
+				<geometry>
+					<mesh filename="package://panel_description/meshes/collisions/Interruptor/Spring.stl" scale="${scale_XYZ} ${scale_XYZ} ${scale_XYZ}"/>
+				</geometry>
+			</collision>
+			<visual>
+				<origin xyz="0 0 0"	rpy="0 0 0"/>
+				<geometry>
+					<mesh filename="package://panel_description/meshes/visual/Interruptor/Spring.stl" scale="${scale_XYZ} ${scale_XYZ} ${scale_XYZ}"/>
+				</geometry>
+			</visual>
+			<inertial>
+				<origin xyz="0 0 0"	rpy="0 0 0"/>
+				<mass value="${springMass}"/>
+				<xacro:cylinder_inertia m="${springMass}" r="${springRadio}" h="${springHeight}" />
+			</inertial>
+		</link>
+		<!-- Spring TO lever JOINT -->
+		<joint name="spring_lever_joint" type="fixed">
+			<parent link="spring_link"/>
+			<child link="lever_link"/>
+			<origin xyz="0 0 0" rpy="0 0 0"/>
+		</joint>
+		<link name='lever_link'>
+			<collision>
+				<origin xyz="0 0 0"	rpy="0 0 0"/>
+				<geometry>
+					<mesh filename="package://panel_description/meshes/collisions/Interruptor/Lever.stl" scale="${scale_XYZ} ${scale_XYZ} ${scale_XYZ}"/>
+				</geometry>
+			</collision>
+			<visual>
+				<origin xyz="0 0 0"	rpy="0 0 0"/>
+				<geometry>
+					<mesh filename="package://panel_description/meshes/visual/Interruptor/Lever.stl" scale="${scale_XYZ} ${scale_XYZ} ${scale_XYZ}"/>
+				</geometry>
+			</visual>
+			<inertial>
+				<origin xyz="0 0 0"	rpy="0 0 0"/>
+				<mass value="${leverMass}"/>
+				<xacro:cylinder_inertia m="${leverMass}" r="${leverRadio}" h="${leverHeight}" />
 			</inertial>
 		</link>
