Commit message: Adding STL switches

File: panel_description/urdf/switch.xacro (robot description, xacro)
@@ -1,10 +1,10 @@
 <?xml version="1.0" ?>
 <robot xmlns:xacro="http://www.ros.org/wiki/xacro">
-	<xacro:macro name="button" params="parent_sector_link child_link x y">
+	<xacro:macro name="switch" params="parent_sector_link child_link x y">
 		<!-- SECTOR_BUTTONS TO CYLINDER JOINT -->
-		<joint name="lid_spring_joint" type="fixed">
+		<joint name="sector_switch_joint" type="fixed">
 			<parent link="${parent_sector_link}"/>
 			<child link="${child_link}"/>
-			<origin xyz="${x} ${y} 0.0" rpy="0 0 ${PI}"/>
+			<origin xyz="${x} ${y} 0.0" rpy="0 0 0"/>
 		</joint>
 		<!-- BUTTON LID -->
@@ -18,5 +18,5 @@
 			<visual>
 				<origin xyz="0 0 0"	rpy="0 0 0"/>
-				<geometry>
+				<geometry>lid
 					<mesh filename="package://panel_description/meshes/visual/lid.stl" scale="${scale_XYZ} ${scale_XYZ} ${scale_XYZ}"/>
 				</geometry>

Commit message: Fix "sector_switch_joint".

File: panel_description/urdf/switch.xacro (robot description, xacro)
@@ -3,5 +3,5 @@
 	<xacro:macro name="switch" params="parent_sector_link child_link x y">
 		<!-- SECTOR_SWITCH TO CYLINDER JOINT -->
-		<joint name="sector_switch_joint" type="fixed">
+		<joint name="switch_joint" type="fixed">
 			<parent link="${parent_sector_link}"/>
 			<child link="${child_link}"/>
