Commit message: Panel switches ya tiene switches

File: panel_description/urdf/sector_switches.xacro (robot description, xacro)
@@ -6,5 +6,5 @@
 			<parent link="base_footprint"/>
 			<child link="sector_switch_link"/>
-			<origin xyz="0 0 0" rpy="0 0 0"/>
+			<origin xyz="0 0 0.3" rpy="0 0 0"/>
 		</joint>
 		<link name="sector_switch_link">
@@ -22,5 +22,5 @@
 			</visual>
 			<inertial>
-				<origin xyz="0 0 0"	rpy="0 0 0"/>switch_1_joint
+				<origin xyz="0 0 0"	rpy="0 0 0"/>
 				<mass value="${switchboxMass}"/>
 				<xacro:box_inertia m="${switchboxMass}" x="${switchboxWidth}" y="${switchboxLength}" z="${switchboxHeight}" />
@@ -28,16 +28,16 @@
 		</link>
 		<!-- Join parts -->
-		<xacro:switch parent_sector_link ="sector_switch_link"  child_link="switch_1_joint" x="0" y="0"/>
-		<!--<xacro:switch parent_sector_link ="sector_switch_link"  child_link= "switch_2_joint" x="0" y="0"/>
-		<xacro:switch parent_sector_link ="sector_switch_link"  child_link= "switch_3_joint" x="0" y="0"/>
-		<xacro:switch parent_sector_link ="sector_switch_link"  child_link= "switch_4_joint" x="0" y="0"/>
-		<xacro:switch parent_sector_link ="sector_switch_link"  child_link= "switch_5_joint" x="0" y="0"/>
-		<xacro:switch parent_sector_link ="sector_switch_link"  child_link= "switch_6_joint" x="0" y="0"/>
-		<xacro:switch parent_sector_link ="sector_switch_link"  child_link= "switch_7_joint" x="0" y="0"/>
-		<xacro:switch parent_sector_link ="sector_switch_link"  child_link= "switch_8_joint" x="0" y="0"/>
-		<xacro:switch parent_sector_link ="sector_switch_link"  child_link= "switch_9_joint" x="0" y="0"/>
-		<xacro:switch parent_sector_link ="sector_switch_link"  child_link= "switch_10_joint" x="0" y="0"/>
-		<xacro:switch parent_sector_link ="sector_switch_link"  child_link= "switch_11_joint" x="0" y="0"/>
-		<xacro:switch parent_sector_link ="sector_switch_link"  child_link= "switch_12_joint" x="0" y="0"/>-->
+		<xacro:switch parent_sector_link ="sector_switch_link"  child_link="switch_1_link" x="0.059" y="0.007" z= "0.034"/>
+		<xacro:switch parent_sector_link ="sector_switch_link"  child_link="switch_2_link" x="0.059" y="0.007" z= "-0.036"/>
+		<xacro:switch parent_sector_link ="sector_switch_link"  child_link="switch_3_link" x="0.059" y="0.007" z= "0.102"/>
+		<xacro:switch parent_sector_link ="sector_switch_link"  child_link="switch_4_link" x="0.059" y="0.007" z= "-0.1053"/>
+		<xacro:switch parent_sector_link ="sector_switch_link"  child_link="switch_5_link" x="0.019" y="0.007" z= "0.034"/>
+		<xacro:switch parent_sector_link ="sector_switch_link"  child_link="switch_6_link" x="0.019" y="0.007" z= "-0.036"/>
+		<xacro:switch parent_sector_link ="sector_switch_link"  child_link="switch_7_link" x="0.019" y="0.007" z= "0.102"/>
+		<xacro:switch parent_sector_link ="sector_switch_link"  child_link="switch_8_link" x="0.019" y="0.007" z= "-0.1053"/>
+		<xacro:switch parent_sector_link ="sector_switch_link"  child_link="switch_9_link" x="-0.021" y="0.007" z= "0.034"/>
+		<xacro:switch parent_sector_link ="sector_switch_link"  child_link="switch_10_link" x="-0.021" y="0.007" z= "-0.036"/>
+		<xacro:switch parent_sector_link ="sector_switch_link"  child_link="switch_11_link" x="-0.021" y="0.007" z= "0.102"/>
+		<xacro:switch parent_sector_link ="sector_switch_link"  child_link="switch_12_link" x="-0.021" y="0.007" z= "-0.1053"/>
 	</xacro:macro>
 </robot>

File: panel_description/urdf/switch.xacro (robot description, xacro)
@@ -1,10 +1,10 @@
 <?xml version="1.0" ?>
 <robot xmlns:xacro="http://www.ros.org/wiki/xacro">
-	<xacro:macro name="switch" params="parent_sector_link child_link x y">
+	<xacro:macro name="switch" params="parent_sector_link child_link x y z">
 		<!-- SECTOR_SWITCH TO CYLINDER JOINT -->
-		<joint name="switch_joint" type="fixed">
+		<joint name="${child_link}_switch_joint" type="fixed">
 			<parent link="${parent_sector_link}"/>
 			<child link="${child_link}"/>
-			<origin xyz="${x} ${y} 0.1" rpy="0 ${PI/2} 0"/>
+			<origin xyz="${x} ${y} ${z}" rpy="${0} ${0} ${PI/2}"/>
 		</joint>
 		<!-- Switch sector LID -->
@@ -29,10 +29,10 @@
 		</link>
 		<!-- Enclosure TO Base1 JOINT -->
-		<joint name="enclosure_base1_joint" type="fixed">
+		<joint name="${child_link}_enclosure_base1_joint" type="fixed">
 			<parent link="${child_link}"/>
-			<child link="base1_link"/>
+			<child link="${child_link}_base1_link"/>
 			<origin xyz="${-0.0125} ${0.01} ${-0.0125}" rpy="0 ${-3*PI/2} ${-PI/2}"/>
 		</joint>
-		<link name='base1_link'>
+		<link name='${child_link}_base1_link'>
 			<collision>
 				<origin xyz="0 0 0"	rpy="0 0 0"/>
@@ -54,10 +54,10 @@
 		</link>
 		<!-- Enclosure TO Base2 JOINT -->
-		<joint name="enclosure_base2_joint" type="fixed">
+		<joint name="${child_link}_enclosure_base2_joint" type="fixed">
 			<parent link="${child_link}"/>
-			<child link="base2_link"/>
+			<child link="${child_link}_base2_link"/>
 			<origin xyz="${-0.0125} ${0.01} 0.01" rpy="0 0 ${-PI/2}"/>
 		</joint>
-		<link name='base2_link'>
+		<link name='${child_link}_base2_link'>
 			<collision>
 				<origin xyz="${-0.01} 0.003 ${-0.005}"	rpy="0 0 0"/>
@@ -79,10 +79,10 @@
 		</link>
 		<!-- Base1 TO triangle JOINT -->
-		<joint name="base1_triangle_joint" type="fixed">
-			<parent link="base1_link"/>
-			<child link="triangle_link"/>
+		<joint name="${child_link}_base1_triangle_joint" type="fixed">
+			<parent link="${child_link}_base1_link"/>
+			<child link="${child_link}_triangle_link"/>
 			<origin xyz="${-0.01} 0.003 ${-0.005}" rpy="0 0 0"/>
 		</joint>
-		<link name='triangle_link'>
+		<link name='${child_link}_triangle_link'>
 			<collision>
 				<origin xyz="0 0 0"	rpy="0 0 0"/>
@@ -104,11 +104,11 @@
 		</link>
 		<!-- Triangle TO trigger JOINT Existe ligera colision con triangle, solo mover x un poquito (+- 0.001)-->
-		<joint name="triangle_trigger_joint" type="revolute">
-			<parent link="triangle_link"/>
-			<child link="trigger_link"/>
+		<joint name="${child_link}_triangle_trigger_joint" type="revolute">
+			<parent link="${child_link}_triangle_link"/>
+			<child link="${child_link}_trigger_link"/>
 			<origin xyz="${-0.005} ${0.015} ${0.005}" rpy="${3*PI/2} ${PI/2} ${PI/2}"/>
 			<limit lower="${-PI/4}" upper="${PI/4}" effort="0" velocity="1"/>
 		</joint>
-		<link name='trigger_link'>
+		<link name='${child_link}_trigger_link'>
 			<collision>
 				<origin xyz="0 0 0"	rpy="0 0 0"/>
@@ -130,10 +130,10 @@
 		</link>
 <!-- Trigger to spring JOINT -->
-		<joint name="trigger_spring_joint" type="fixed">
-			<parent link="trigger_link"/>
-			<child link="spring_link"/>
+		<joint name="${child_link}_trigger_spring_joint" type="fixed">
+			<parent link="${child_link}_trigger_link"/>
+			<child link="${child_link}_spring_link"/>
 			<origin xyz="0 0 0" rpy="0 0 0"/>
 		</joint>
-		<link name='spring_link'>
+		<link name='${child_link}_spring_link'>
 			<collision>
 				<origin xyz="0 0 0"	rpy="0 0 0"/>
@@ -155,10 +155,10 @@
 		</link>
 		<!-- Spring TO lever JOINT -->
-		<joint name="spring_lever_joint" type="fixed">
-			<parent link="spring_link"/>
-			<child link="lever_link"/>
+		<joint name="${child_link}_spring_lever_joint" type="fixed">
+			<parent link="${child_link}_spring_link"/>
+			<child link="${child_link}_lever_link"/>
 			<origin xyz="0 0 0" rpy="0 0 0"/>
 		</joint>
-		<link name='lever_link'>
+		<link name='${child_link}_lever_link'>
 			<collision>
 				<origin xyz="0 0 0"	rpy="0 0 0"/>
